File: agat_disk_adapter.kicad_pcb (KiCad board)
At the start: 2 copper layers, 53.3 x 61 mm, 14 parts, among them J1 КОНТРОЛЛЕР, J2_A1 ИЗОТ, J2_B2 ИЗОТ, J3 DISK II, J4 GOTEK, J5 Питание GOTEK, J6 ВБ, J7 Джамперы, J8 ВБ2, J9 PIN_32, J9_A1 КОНТРОЛЛЕР, J9_B2 КОНТРОЛЛЕР

Commit message: advance
Parts:
- moved J5 0.64 mm to (45.7, 87.0)
Connections:
- net /PIN_32 renamed /G32
- J1 pad 14: /EN1 -> /DE1
- J2_B2 pad 7: /EN_J2 -> /DE_J2
- J3 pad 14: /EN_J3 -> /DE_J3
- J4 pad 10: /EN_J4 -> /DE_J4
- J6 pad 1: /EN_J2 -> /DE_J2
- J6 pad 10: /EN_J4 -> /DE2
- J6 pad 2: /EN_J2 -> /DE2
- J6 pad 4: /EN2 -> GND
- J6 pad 5: /EN_J3 -> /DE_J3
- J6 pad 6: /EN_J3 -> /DE2
- J6 pad 8: /EN2 -> /+5
- J6 pad 9: /EN_J4 -> /DE_J4
- J8 pad 1: /DS2 -> /DE2
- J9_B2 pad 7: /EN1 -> /DE1
Routing:
- net /EN_J3: track 167.5 -> 0.00 mm
- net /DE_J3: track 0.00 -> 167.5 mm
- net /EN1: track 145.9 -> 83.8 mm
- net /DE1: track 0.00 -> 62.1 mm
- net /EN_J2: track 38.6 -> 0.00 mm
- net /DE_J2: track 0.00 -> 38.6 mm
- net /EN_J4: track 26.6 -> 0.00 mm
- net /DE_J4: track 0.00 -> 26.6 mm
- net /+12: track 7.66 -> 2.36 mm
- net /-12: track 29.1 -> 29.8 mm
