File: agat_disk_adapter.kicad_sch (KiCad schematic)
At the start: 14 parts, among them J1 КОНТРОЛЛЕР, J2_A1 ИЗОТ, J2_B2 ИЗОТ, J3 DISK II, J4 GOTEK, J5 Питание GOTEK, J6 ВБ, J7 Джамперы, J8 ВБ2, J9 PIN_32, J9_A1 КОНТРОЛЛЕР, J9_B2 КОНТРОЛЛЕР

Commit message: advance
Connections:
- net +5: now also J6.8 (Pin_8)
- net DE2: now also J6.10 (Pin_10), J6.2 (Pin_2), J6.6 (Pin_6)
- net EN1: no longer J1.14 (Pin_14), J9_B2.7 (Pin_7)
- net GND: now also J6.4 (Pin_4)
- removed net EN2: J6.4 (Pin_4), J6.8 (Pin_8)
- net EN_J2 renamed DE_J2
- net DE_J2: no longer J6.2 (Pin_2)
- net EN_J3 renamed DE_J3
- net DE_J3: no longer J6.6 (Pin_6)
- net EN_J4 renamed DE_J4
- net DE_J4: no longer J6.10 (Pin_10)
- net PIN_32 renamed G32
- new net DE1: J1.14 (Pin_14), J9_B2.7 (Pin_7)
Other:
- moved on the sheet: J6
Changed lines of the file:
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@@
 	)
 	(junction
+		(at 50.8 115.57)
+		(diameter 0)
+		(color 0 0 0 0)
+	)
+	(junction
 		(at 73.66 106.68)
 		(diameter 0)
@@
 	(wire
 		(pts
-			(xy 41.91 109.855) (xy 50.165 109.855)
+			(xy 41.91 110.49) (xy 50.8 110.49)
 		)
 		(stroke
@@
 	(wire
 		(pts
-			(xy 52.07 105.41) (xy 52.07 114.935)
-		)
-		(stroke
-			(width 0)
-			(type default)
-		)
-	)
-	(wire
-		(pts
 			(xy 73.66 86.36) (xy 76.2 86.36)
 		)
@@
 	(wire
 		(pts
-			(xy 50.165 112.395) (xy 50.165 117.475)
-		)
-		(stroke
-			(width 0)
-			(type default)
-		)
-	)
-	(wire
-		(pts
 			(xy 83.82 86.36) (xy 83.82 106.68)
 		)
@@
 	(wire
 		(pts
-			(xy 19.05 105.41) (xy 52.07 105.41)
-		)
-		(stroke
-			(width 0)
-			(type default)
-		)
-	)
-	(wire
-		(pts
 			(xy 93.98 154.305) (xy 93.98 161.925)
 		)
@@
 	(wire
 		(pts
-			(xy 19.05 114.935) (xy 19.05 105.41)
-		)
-		(stroke
-			(width 0)
-			(type default)
-		)
-	)
-	(wire
-		(pts
 			(xy 81.28 119.38) (xy 81.28 127)
 		)
@@
 	(wire
 		(pts
-			(xy 20.955 109.855) (xy 29.21 109.855)
-		)
-		(stroke
-			(width 0)
-			(type default)
-		)
-	)
-	(wire
-		(pts
 			(xy 76.2 119.38) (xy 76.2 127)
 		)
@@
 	(wire
 		(pts
-			(xy 20.955 109.855) (xy 20.955 107.315)
-		)
-		(stroke
-			(width 0)
-			(type default)
-		)
-	)
-	(wire
-		(pts
 			(xy 106.68 180.34) (xy 106.68 175.26)
 		)
@@
 	(wire
 		(pts
-			(xy 20.955 117.475) (xy 29.21 117.475)
+			(xy 20.955 118.11) (xy 29.21 118.11)
 		)
 		(stroke
@@
 	(wire
 		(pts
-			(xy 91.44 38.1) (xy 93.98 38.1)
+			(xy 50.8 115.57) (xy 50.8 120.65)
 		)
 		(stroke
@@
 	(wire
 		(pts
-			(xy 81.28 18.415) (xy 81.28 25.4)
+			(xy 91.44 38.1) (xy 93.98 38.1)
 		)
 		(stroke
@@
 	(wire
 		(pts
-			(xy 50.165 122.555) (xy 50.165 120.015)
+			(xy 81.28 18.415) (xy 81.28 25.4)
 		)
 		(stroke
@@
 	(wire
 		(pts
-			(xy 20.955 107.315) (xy 50.165 107.315)
-		)
-		(stroke
-			(width 0)
-			(type default)
-		)
-	)
-	(wire
-		(pts
 			(xy 73.66 66.675) (xy 73.66 73.66)
 		)
@@
 	(wire
 		(pts
-			(xy 20.955 112.395) (xy 29.21 112.395)
+			(xy 20.955 113.03) (xy 29.21 113.03)
 		)
 		(stroke
@@
 	(wire
 		(pts
-			(xy 41.91 112.395) (xy 50.165 112.395)
+			(xy 41.91 113.03) (xy 48.26 113.03)
 		)
 		(stroke
@@
 	(wire
 		(pts
+			(xy 50.8 110.49) (xy 50.8 115.57)
+		)
+		(stroke
+			(width 0)
+			(type default)
+		)
+	)
+	(wire
+		(pts
 			(xy 91.44 119.38) (xy 91.44 127)
 		)
@@
 	(wire
 		(pts
-			(xy 20.955 120.015) (xy 29.21 120.015)
+			(xy 22.86 120.65) (xy 29.21 120.65)
 		)
 		(stroke
@@
 	(wire
 		(pts
-			(xy 41.91 114.935) (xy 52.07 114.935)
+			(xy 41.91 115.57) (xy 50.8 115.57)
 		)
 		(stroke
@@
 	(wire
 		(pts
+			(xy 22.86 110.49) (xy 29.21 110.49)
+		)
+		(stroke
+			(width 0)
+			(type default)
+		)
+	)
+	(wire
+		(pts
 			(xy 71.12 133.985) (xy 71.12 141.605)
 		)
@@
 	(wire
 		(pts
-			(xy 20.955 112.395) (xy 20.955 117.475)
+			(xy 20.955 113.03) (xy 20.955 118.11)
 		)
 		(stroke
@@
 	(wire
 		(pts
-			(xy 19.05 114.935) (xy 29.21 114.935)
+			(xy 22.86 115.57) (xy 29.21 115.57)
 		)
 		(stroke
@@
 	(wire
 		(pts
-			(xy 50.165 107.315) (xy 50.165 109.855)
-		)
-		(stroke
-			(width 0)
-			(type default)
-		)
-	)
-	(wire
-		(pts
 			(xy 95.885 191.643) (xy 93.98 191.643)
 		)
@@
 	(wire
 		(pts
-			(xy 20.955 122.555) (xy 50.165 122.555)
-		)
-		(stroke
-			(width 0)
-			(type default)
-		)
-	)
-	(wire
-		(pts
 			(xy 73.66 141.605) (xy 76.2 141.605)
 		)
@@
 	(wire
 		(pts
-			(xy 41.91 117.475) (xy 50.165 117.475)
+			(xy 41.91 118.11) (xy 48.26 118.11)
 		)
 		(stroke
@@
 	(wire
 		(pts
-			(xy 20.955 120.015) (xy 20.955 122.555)
-		)
-		(stroke
-			(width 0)
-			(type default)
-		)
-	)
-	(wire
-		(pts
 			(xy 81.28 38.1) (xy 81.28 73.66)
 		)
@@
 	(wire
 		(pts
-			(xy 41.91 120.015) (xy 50.165 120.015)
+			(xy 41.91 120.65) (xy 50.8 120.65)
 		)
 		(stroke
@@
 		)
 	)
-	(label "EN_J4"
-		(at 22.86 120.015 0)
+	(label "DE_J4"
+		(at 22.86 120.65 0)
 		(effects
 			(font
@@
 		)
 	)
-	(label "EN2"
-		(at 48.26 117.475 180)
+	(label "+5"
+		(at 48.26 118.11 180)
 		(effects
 			(font
@@
 		)
 	)
-	(label "EN_J3"
+	(label "DE_J3"
 		(at 78.74 161.925 90)
 		(effects
@@
 		)
 	)
-	(label "EN2"
-		(at 48.26 112.395 180)
+	(label "GND"
+		(at 48.26 113.03 180)
 		(effects
 			(font
@@
 		)
 	)
-	(label "PIN_32"
+	(label "G32"
 		(at 91.948 175.26 0)
 		(effects
@@
 		)
 	)
-	(label "EN1"
+	(label "DE1"
 		(at 78.74 66.675 270)
 		(effects
@@
 		)
 	)
-	(label "EN_J2"
-		(at 48.26 109.855 180)
+	(label "DE2"
+		(at 48.26 110.49 180)
 		(effects
 			(font
@@
 		)
 	)
-	(label "EN1"
+	(label "DE1"
 		(at 78.74 127 90)
 		(effects
@@
 		)
 	)
-	(label "EN_J2"
+	(label "DE_J2"
 		(at 78.74 18.415 270)
 		(effects
@@
 		)
 	)
-	(label "EN_J2"
-		(at 22.86 109.855 0)
+	(label "DE_J2"
+		(at 22.86 110.49 0)
 		(effects
 			(font
@@
 	)
 	(label "EN1"
-		(at 22.86 112.395 0)
+		(at 22.86 113.03 0)
 		(effects
 			(font
@@
 		)
 	)
-	(label "EN_J4"
-		(at 48.26 120.015 180)
+	(label "DE2"
+		(at 48.26 120.65 180)
 		(effects
 			(font
@@
 		)
 	)
-	(label "EN_J3"
-		(at 48.26 114.935 180)
+	(label "DE2"
+		(at 48.26 115.57 180)
 		(effects
 			(font
@@
 		)
 	)
-	(label "EN_J3"
-		(at 22.86 114.935 0)
+	(label "DE_J3"
+		(at 22.86 115.57 0)
 		(effects
 			(font
@@
 	)
 	(label "EN1"
-		(at 22.86 117.475 0)
+		(at 22.86 118.11 0)
 		(effects
 			(font
@@
 		)
 	)
-	(label "EN_J4"
+	(label "DE_J4"
 		(at 63.5 170.18 270)
 		(effects
@@
 	(symbol
 		(lib_id "Connector_Generic:Conn_02x05_Odd_Even")
-		(at 34.29 114.935 0)
+		(at 34.29 115.57 0)
 		(unit 1)
 		(body_style 1)
@@
 		(dnp no)
 		(property "Reference" "J6"
-			(at 35.56 103.505 0)
+			(at 35.56 106.934 0)
 			(show_name no)
 			(do_not_autoplace no)
@@
 		)
 		(property "Value" "ВБ"
-			(at 35.56 100.965 0)
+			(at 35.56 104.394 0)
 			(show_name no)
 			(do_not_autoplace no)
@@
 		)
 		(property "Footprint" "Connector_IDC:IDC-Header_2x05_P2.54mm_Vertical"
-			(at 34.29 114.935 0)
+			(at 34.29 115.57 0)
 			(hide yes)
 			(show_name no)
@@
 		)
 		(property "Datasheet" ""
-			(at 34.29 114.935 0)
+			(at 34.29 115.57 0)
 			(hide yes)
 			(show_name no)
@@
 		)
 		(property "Description" "Generic connector, double row, 02x05, odd/even pin numbering scheme (row 1 odd numbers, row 2 even numbers), script generated (kicad-library-utils/schlib/autogen/connector/)"
-			(at 34.29 114.935 0)
+			(at 34.29 115.57 0)
 			(hide yes)
 			(show_name no)
